Commit message: Update robot.urdf
in progress

File: robot_description/urdf/robot.urdf (robot description, URDF)
Before this commit: robot my_robot, 4 links, 3 joints
Links:
- added link caster_wheel; visual sphere radius=0.01
Joints:
- added joint caster_wheel_joint: type fixed, parent chassis, child caster_wheel, origin xyz=-0.01 -0.02 -0.01 rpy=0.0 0.0 0.0

Commit message: Update robot.urdf
edit camera

File: robot_description/urdf/robot.urdf (robot description, URDF)
Before this commit: robot my_robot, 5 links, 4 joints
Links:
- added link camera; visual box size=0.02 0.02 0.02
- added link lidar; visual cylinder length=0.010 radius=0.018
- link caster_wheel: geometry visual sphere radius=0.015
Joints:
- added joint camera_joint: type fixed, parent chassis, child camera, origin xyz=0.021 0.0 0.011 rpy=0.0 0.0 0.0
- added joint lidar_joint: type fixed, parent chassis, child lidar, origin xyz=-0.010 0.0 0.011 rpy=0.0 0.0 0.0
- joint caster_wheel_joint: origin xyz=-0.01 -0.02 -0.01 rpy=0.0 0.0 0.0 -> xyz=0.0 0.0 0.0 rpy=0.0 0.0 0.0

Commit message: Update robot.urdf
Add <collision>

File: robot_description/urdf/robot.urdf (robot description, URDF)
Before this commit: robot my_robot, 7 links, 6 joints
Links:
- link camera: geometry collision box size=0.02 0.02 0.02; visual box size=0.02 0.02 0.02
- link caster_wheel: geometry collision sphere radius=0.015; visual sphere radius=0.015
- link chassis: geometry collision box size=0.10 0.065 0.03; visual box size=0.10 0.065 0.03
- link left_wheel: geometry collision cylinder length=0.010 radius=0.018; visual cylinder length=0.010 radius=0.018
- link lidar: geometry collision cylinder length=0.010 radius=0.018; visual cylinder length=0.010 radius=0.018
- link right_wheel: geometry collision cylinder length=0.010 radius=0.018; visual cylinder length=0.010 radius=0.018

Commit message: Update robot.urdf
add inertial tags

File: robot_description/urdf/robot.urdf (robot description, URDF)
Before this commit: robot my_robot, 7 links, 6 joints
Links:
- link camera: mass None -> 0.02
- link chassis: mass None -> 0.05
- link left_wheel: mass None -> 0.02
- link lidar: mass None -> 0.02
- link right_wheel: mass None -> 0.02
